Commit message: Revert "Final2"
This reverts commit 772941d61b31ec51b17a83efbe9fb5629372486f.

File: clover_description/urdf/clover/clover4_base.xacro (robot description, xacro)
@@ -21,5 +21,5 @@
   </xacro:if>
   <!-- Gazebo plugins -->
-  <xacro:include filename="$(find drone_description)/urdf/clover/clover4_gazebo.xacro" />
+  <xacro:include filename="$(find clover_description)/urdf/clover/clover4_gazebo.xacro" />
   <xacro:if value="$(arg enable_logging)">
     <!-- Instantiate a logger -->

File: clover_description/urdf/clover/clover4_macros.xacro (robot description, xacro)
@@ -48,5 +48,5 @@
         <geometry>
           <!-- Note: Texture files are expected to be in the same directory as the model -->
-          <mesh filename="package://drone_description/meshes/clover4/clover_body_solid.dae"
+          <mesh filename="package://clover_description/meshes/clover4/clover_body_solid.dae"
             scale="1 1 1"/>
         </geometry>
@@ -106,5 +106,5 @@
         <origin xyz="0 0 0.025" rpy="0 0 0"/>
         <geometry>
-          <mesh filename="package://drone_description/meshes/clover4/clover_guards_transparent.dae"
+          <mesh filename="package://clover_description/meshes/clover4/clover_guards_transparent.dae"
             scale="1 1 1"/>
         </geometry>
@@ -177,5 +177,5 @@
       <visual>
         <geometry>
-          <mesh filename="package://drone_description/meshes/${mesh}"
+          <mesh filename="package://clover_description/meshes/${mesh}"
             scale="1 1 1" />
         </geometry>
